File: switch.kicad_sch (KiCad schematic)
At the start: 4 parts, among them K2 Relay_SPDT, U22 LTV-817

Commit message: idk
Parts:
- added J5: Conn_01x06_Pin, symbol Connector:Conn_01x06_Pin
Changed lines of the file:
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@@
+	)
+	(symbol
+		(lib_id "Connector:Conn_01x06_Pin")
+		(at 83.82 74.93 0)
+		(unit 1)
+		(exclude_from_sim no)
+		(in_bom yes)
+		(on_board yes)
+		(dnp no)
+		(fields_autoplaced yes)
+		(property "Reference" "J5"
+			(at 84.455 64.77 0)
+			(effects
+				(font
+					(size 1.27 1.27)
+				)
+			)
+		)
+		(property "Value" "Conn_01x06_Pin"
+			(at 84.455 67.31 0)
+			(effects
+				(font
+					(size 1.27 1.27)
+				)
+			)
+		)
+		(property "Footprint" ""
+			(at 83.82 74.93 0)
+			(effects
+				(font
+					(size 1.27 1.27)
+				)
+				(hide yes)
+			)
+		)
+		(property "Datasheet" "~"
+			(at 83.82 74.93 0)
+			(effects
+				(font
+					(size 1.27 1.27)
+				)
+				(hide yes)
+			)
+		)
+		(property "Description" "Generic connector, single row, 01x06, script generated"
+			(at 83.82 74.93 0)
+			(effects
+				(font
+					(size 1.27 1.27)
+				)
+				(hide yes)
+			)
+		)
+		(pin "3"
+		)
+		(pin "2"
+		)
+		(pin "1"
+		)
+		(pin "6"
+		)
+		(pin "5"
+		)
+		(pin "4"
+		)
+		(instances
+			(project ""
+				(path "/ea916249-dd1d-4e08-8738-941d6aac22ff/0fcd6b21-2536-4892-87a9-4a6d6c328fb0/b7ab99f2-8081-4344-be8a-8175e61b238e"
+					(reference "J13")
+					(unit 1)
+				)
+				(path "/ea916249-dd1d-4e08-8738-941d6aac22ff/0fcd6b21-2536-4892-87a9-4a6d6c328fb0/db85d050-314d-4706-8d05-898dffc558fc"
+					(reference "J14")
+					(unit 1)
+				)
+				(path "/ea916249-dd1d-4e08-8738-941d6aac22ff/2e7bd37d-1784-4969-9b01-14f1ff8ed01f/b7ab99f2-8081-4344-be8a-8175e61b238e"
+					(reference "J8")
+					(unit 1)
+				)
+				(path "/ea916249-dd1d-4e08-8738-941d6aac22ff/2e7bd37d-1784-4969-9b01-14f1ff8ed01f/db85d050-314d-4706-8d05-898dffc558fc"
+					(reference "J9")
+					(unit 1)
+				)
+				(path "/ea916249-dd1d-4e08-8738-941d6aac22ff/97ba9808-3c28-4872-985a-94496d356f3f/b7ab99f2-8081-4344-be8a-8175e61b238e"
+					(reference "J7")
+					(unit 1)
+				)
+				(path "/ea916249-dd1d-4e08-8738-941d6aac22ff/97ba9808-3c28-4872-985a-94496d356f3f/db85d050-314d-4706-8d05-898dffc558fc"
+					(reference "J5")
+					(unit 1)
+				)
+			)
+		)
 	)
 	(symbol
